File: hardware/carrier-board/carrier-board.kicad_sch (KiCad schematic)
At the start: 0 parts

Commit message: Resolve connector and clock synthesizer parts; drop 4th input sheet
Connector: confirmed exact Samtec part numbers directly from Trenz's
own "5.2 x 7.6 SoM ST5 and SS5 B2B Connectors" page, cross-referenced
against Samtec's catalog -- carrier-side socket is SS5-80-3.50-L-D-K-TR
(Trenz ref REF-192552-01), 160-position/3.5mm stack height, matching
TE0807's onboard ST5 (REF-192552-02). KiCad footprint/symbol/3D model
available from the official KiCad footprint library and SnapEDA --
nothing to hand-build.

Clock synthesizer: selected Silicon Labs Si5341A, a 10-output
any-frequency clock generator explicitly referenced in Silicon Labs' own
timing reference designs for Kintex/Virtex UltraScale GTH transceiver
applications. One chip feeds all 4 quads' reference pins independently
(no sharing, per the corrected clocking conclusion), with 6 outputs
spare for future genlock/reference distribution needs.

Also fixed the KiCad skeleton to match the finalized 3-in+1-out scope:
removed hdmi_in4.kicad_sch and its sheet symbol (this board doesn't have
a 4th input -- that's deferred to a second board), re-validated via
kicad-cli sch upgrade (clean round-trip) and sch erc (0 violations
across the remaining 8 sheets), and updated the title-block comment.

Updated carrier-board-spec.md and the KiCad README to match throughout.
Other:
- removed sheet HDMI Input 4
Changed lines of the file:
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@@
 		(company "OpenAVSwitch")
 		(comment 1 "SOM+carrier for Trenz TE0807 (XCZU7EV) -- see docs/carrier-board-spec.md")
-		(comment 2 "3 native in + 1 native out fit (1 quad each, no sharing); 4th input needs a decision")
+		(comment 2 "3 native HDMI in + 1 native out, 1 GTH quad each, no sharing. 4th input on a 2nd board.")
 	)
 	(sheet
@@
 			(show_name no)
 			(do_not_autoplace no)
-			(effects
-				(font
-					(size 1.27 1.27)
-				)
-				(justify left top)
-			)
-		)
-	)
-	(sheet
-		(at 20 120)
-		(size 25.4 12.7)
-		(exclude_from_sim no)
-		(in_bom yes)
-		(on_board yes)
-		(dnp no)
-		(fields_autoplaced yes)
-		(stroke
-			(width 0.1524)
-			(type solid)
-		)
-		(fill
-			(color 0 0 0 0)
-		)
-		(property "Sheetname" "HDMI Input 4"
-			(at 20 119 0)
-			(show_name no)
-			(do_not_autoplace no)
-			(effects
-				(font
-					(size 1.27 1.27)
-				)
-				(justify left bottom)
-			)
-		)
-		(property "Sheetfile" "hdmi_in4.kicad_sch"
-			(at 20 134 0)
-			(show_name no)
-			(do_not_autoplace no)
