File: hardware/carrier-board/clocking.kicad_sch (KiCad schematic)
At the start: 0 parts

Commit message: Transcribe Si5341A and generic HDMI connector; ESD8040 genuinely blocked
Si5341A-B-GM: hand-transcribed all 64 QFN pins from Silicon Labs'
primary Si5341/40 Data Sheet (Table 17), reached via pdftotext after
several blocked/wrong-document fetch attempts on adjacent URLs.
Cross-checked the extraction sums to exactly 64 pins with no gaps or
duplicates before trusting it. Footprint matched to KiCad's own
standard JEDEC MO-220 QFN-64-1EP_9x9mm_P0.5mm_EP5.2x5.2mm library part,
verified against the datasheet's own Table 18 package dimensions and
copied in from the local KiCad install rather than hand-authored.
Placed in clocking.kicad_sch; validated clean on the first kicad-cli
attempt (single-unit symbol design avoided the SS5 connector's
multi-unit quirk entirely).

HDMI connector: caught that "Amphenol GSD1S211-K1E1-4030" (named in an
earlier research pass) never turns up anywhere in search -- treating it
as an unverified/likely-fabricated part number rather than building on
it further. Built a generic HDMI_TypeA_Receptacle symbol instead from
the public HDMI specification's pinout (manufacturer-independent, so
high confidence for the electrical pinout specifically). No footprint
assigned -- a real manufacturer part still needs picking before layout.

ESD8040: genuinely could not get the pin table after 5+ attempts across
onsemi.com (403), Mouser/Farnell (timeout, or once returned an unrelated
part's datasheet -- ESD8351 -- caught via pdfinfo's Title field before
it got used), DigiKey (410 Gone), and web archive (blocked entirely).
Not fabricated as a workaround -- documented as blocked in both
carrier-board-spec.md and the KiCad README.

Corrected the connector part-number claim in carrier-board-spec.md,
updated the KiCad README with full current status.
Parts:
- added U1: Si5341A-B-GM, carrier_footprints:QFN-64-1EP_9x9mm_P0.5mm_EP5.2x5.2mm, symbol Si5341A-B-GM:Si5341A-B-GM
Changed lines of the file:
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@@
 		(title "OpenAVSwitch Carrier Board - Reference Clocking")
 		(company "OpenAVSwitch")
-		(comment 1 "Stub sheet -- not yet populated, see docs/carrier-board-spec.md")
+		(comment 1 "Si5341A placed (10-output any-frequency generator, 4 outputs used: quads 224/225/226/227).")
+	)
+	(symbol
+		(lib_id "Si5341A-B-GM:Si5341A-B-GM")
+		(at 99.06 99.06 0)
+		(unit 1)
+		(body_style 1)
+		(exclude_from_sim no)
+		(in_bom yes)
+		(on_board yes)
+		(in_pos_files yes)
+		(dnp no)
+		(property "Reference" "U1"
+			(at 99.06 55 0)
+			(show_name no)
+			(do_not_autoplace no)
+			(effects
+				(font
+					(size 1.27 1.27)
+				)
+			)
+		)
+		(property "Value" "Si5341A-B-GM"
+			(at 99.06 145 0)
+			(show_name no)
+			(do_not_autoplace no)
+			(effects
+				(font
+					(size 1.27 1.27)
+				)
+			)
+		)
+		(property "Footprint" "carrier_footprints:QFN-64-1EP_9x9mm_P0.5mm_EP5.2x5.2mm"
+			(at 99.06 99.06 0)
+			(hide yes)
+			(show_name no)
+			(do_not_autoplace no)
+			(effects
+				(font
+					(size 1.27 1.27)
+				)
+			)
+		)
+		(property "Datasheet" ""
+			(at 99.06 99.06 0)
+			(show_name no)
+			(do_not_autoplace no)
+			(effects
+				(font
+					(size 1.27 1.27)
+				)
+			)
+		)
+		(property "Description" ""
+			(at 99.06 99.06 0)
+			(show_name no)
+			(do_not_autoplace no)
+			(effects
+				(font
+					(size 1.27 1.27)
+				)
+			)
+		)
+		(pin "1"
+		)
+		(pin "2"
+		)
+		(pin "3"
+		)
+		(pin "4"
+		)
+		(pin "5"
+		)
+		(pin "6"
+		)
+		(pin "7"
+		)
+		(pin "8"
+		)
+		(pin "9"
+		)
+		(pin "10"
+		)
+		(pin "11"
+		)
+		(pin "12"
+		)
+		(pin "13"
+		)
+		(pin "14"
+		)
+		(pin "15"
+		)
+		(pin "16"
+		)
+		(pin "17"
+		)
+		(pin "18"
+		)
+		(pin "19"
+		)
+		(pin "20"
+		)
+		(pin "21"
+		)
+		(pin "22"
+		)
+		(pin "23"
+		)
+		(pin "24"
+		)
+		(pin "25"
+		)
+		(pin "26"
+		)
+		(pin "27"
+		)
+		(pin "28"
+		)
+		(pin "29"
+		)
+		(pin "30"
+		)
+		(pin "31"
+		)
+		(pin "32"
+		)
+		(pin "33"
+		)
+		(pin "34"
+		)
+		(pin "35"
+		)
+		(pin "36"
+		)
+		(pin "37"
+		)
+		(pin "38"
+		)
+		(pin "39"
+		)
+		(pin "40"
+		)
+		(pin "41"
+		)
+		(pin "42"
+		)
+		(pin "43"
+		)
+		(pin "44"
+		)
+		(pin "45"
+		)
+		(pin "46"
+		)
+		(pin "47"
+		)
+		(pin "48"
+		)
+		(pin "49"
+		)
+		(pin "50"
+		)
+		(pin "51"
+		)
+		(pin "52"
+		)
+		(pin "53"
+		)
+		(pin "54"
+		)
+		(pin "55"
+		)
+		(pin "56"
+		)
+		(pin "57"
+		)
+		(pin "58"
+		)
+		(pin "59"
+		)
+		(pin "60"
+		)
+		(pin "61"
+		)
+		(pin "62"
+		)
+		(pin "63"
+		)
+		(pin "64"
+		)
 	)
 	(sheet_instances
