File: hardware/carrier-board/som_connector.kicad_sch (KiCad schematic)
At the start: 0 parts

Commit message: Integrate real downloaded component libraries; place first symbols
User downloaded SnapEDA exports for TXS0102DCUR and SS5-80-3.50-L-D-K-TR
(the level translator and SOM B2B connector selected in
carrier-board-spec.md). Extracted into hardware/carrier-board/libs/
(symbols, footprints, STEP models), re-validated every symbol and
footprint through kicad-cli sym/fp upgrade before trusting them, and
wired them into the project via sym-lib-table/fp-lib-table (with
name-aliased footprint entries matching what's baked into each
downloaded symbol's Footprint property).

Placed TXS0102DCUR in all 4 relevant sheets (hdmi_in1-3, hdmi_out) --
caught and fixed a real bug in the process (nested sub-symbol name
needs the bare "PART_0_0" form, not "LIB:PART_0_0" -- the first attempt
failed to load entirely). Also fixed grid-off-placement and a
lib_symbol_mismatch (embedded copies were missing several properties
present in the source library) once ERC surfaced them. Full-hierarchy
ERC now shows only expected "pin not connected" warnings across all
4 sheets -- correct for placed-but-unwired components, no structural
errors.

Placed J1 of the SS5 connector (160 pins, 2-unit symbol) in
som_connector.kicad_sch. Hit a real, narrower limit here: kicad-cli's
non-interactive upgrade collapses both unit instances to "unit 1"
during normalization. Verified this doesn't lose or duplicate any pin
data (160 unique pins, correctly mapped) -- it's a cosmetic/organizational
quirk in headless multi-unit handling, not a netlist bug -- but
couldn't resolve it further without the interactive GUI's purpose-built
multi-unit placement tools. Flagged in the README for the user to check
in real KiCad before J2-J4 get placed the same way.

Si5341A, ESD8040, and the Amphenol HDMI connector still need
hand-transcription from datasheets -- no pre-made libraries found for
those. README updated with full current status and next steps.
Parts:
- added J1 (x2): SS5-80-3.50-L-D-K-TR, SS5-80-3.50-X-D-K-XX:SAMTEC_SS5-80-3.50-X-D-K-XX, symbol SS5-80-3.50-X-D-K-XX:SS5-80-3.50-X-D-K-XX
Other:
- title: OpenAVSwitch Carrier Board - SOM Connector (Trenz TE0807 B2B x4) -> OpenAVSwitch Carrier Board - SOM Connector

Commit message: Place J2-J4; correct a real bug in the earlier "cosmetic quirk" finding
Placed all 3 remaining SOM connectors (J1 already done) using the same
pattern. While verifying, found the earlier assessment of the J1
"multi-unit quirk" was wrong in an important way: it wasn't just the
unit field collapsing to 1 (cosmetic), it also ballooned each instance
from its correct 80 pins to all 160 -- a real duplication, not a
labeling issue.

Traced the root cause by regenerating from scratch and checking pin
data before vs. after kicad-cli sch upgrade: correct (80 pins/unit,
properly split 1-80 / 81-160) immediately after generation, corrupted
(160 pins/unit, different_unit_net ERC errors) only after running
upgrade on the file. kicad-cli's non-interactive upgrade actively
corrupts multi-unit symbol instances -- it's not a preservation issue,
it's the thing causing the damage.

Fix: never run sch upgrade on files with multi-unit symbol instances;
validate with sch erc alone, which is read-only and reports correctly
(confirmed via diff that erc doesn't modify the file). Regenerated
som_connector.kicad_sch clean with J1-J4 all correctly split 80/80,
verified via erc only -- zero different_unit_net violations, only the
expected unconnected-pin warnings.

This resolves what was previously flagged as needing a GUI check in
real KiCad -- it didn't need one, the data was always fine once the
corrupting command is avoided. Updated the README to explain the actual
root cause instead of the wrong "cosmetic, GUI-verify" framing, and
noted a genuinely cosmetic (not correctness) item: J2-J4 sit beyond a
single A4 page's visible bounds given each connector's ~200mm pin
column height.
Parts:
- removed J1 (x2): SS5-80-3.50-L-D-K-TR, SS5-80-3.50-X-D-K-XX:SAMTEC_SS5-80-3.50-X-D-K-XX, symbol SS5-80-3.50-X-D-K-XX:SS5-80-3.50-X-D-K-XX
- added J1, J2, J3, J4: SS5-80-3.50-L-D-K-TR, SS5-80-3.50-X-D-K-XX:SAMTEC_SS5-80-3.50-X-D-K-XX, symbol SS5-80-3.50-X-D-K-XX:SS5-80-3.50-X-D-K-XX
