File: hardware/carrier-board/power.kicad_sch (KiCad schematic)
At the start: 0 parts

Commit message: Draw the power-good sequencing circuit in power.kicad_sch
Schematic-captured the wired-AND circuit already fully specified in
carrier-board-spec.md: 7 PG_* signals from the TE0807 TRM's Table 18,
3 pull-up resistors (10k to +3V3) for the ones needing carrier-provided
pull-ups, and an R4/C1 debounce filter producing VCCO_EN for whichever
VCCO regulator gets chosen later.

Used KiCad's standard Device:R/Device:C symbols rather than anything
transcribed. Represented the "these 7 differently-named signals are
electrically one node" requirement using same-text label coincidence
(global label for the real signal name + local label "PWR_GOOD_ALL" at
the identical coordinate) instead of hand-routed bus wires with
T-junctions -- avoids a whole class of wire-endpoint-math mistakes.

Hit and fixed a real bug along the way: an earlier version routed a
pull-up resistor's two ends to labels via wires, and ended up shorting
+3V3 directly to the sense node on one resistor (a coordinate-math
error, caught by kicad-cli sch erc's multiple_net_names check flagging
+3V3 merged with PWR_GOOD_ALL directly). Rebuilt using the label-
coincidence approach specifically to eliminate that bug class, then
re-verified erc shows only the two *intended* warnings (the deliberate
label merge, and VCCO_EN's expected single-consumer state since no
regulator exists yet).

Also fixed grid-off-placements and added a missing Device library
entry to sym-lib-table (using the portable ${KICAD10_SYMBOL_DIR}
variable, matching KiCad's own template rather than a hardcoded path).

Confirmed sch upgrade is safe for this file (single-unit R/C symbols
only, unlike the multi-unit SS5 connector) -- pin count unchanged
before/after.
Parts:
- added C1: 100nF, symbol Device:C
- added R1, R2, R3: 10k, symbol Device:R
- added R4: 1k, symbol Device:R
Connections:
- new net +3V3: R1.2, R2.2, R3.2
- new net GND: C1.1
- new net LP_GOOD: C1.2, R1.1, R2.1, R3.1, R4.1, R4.2
Other:
- title: OpenAVSwitch Carrier Board - Power (carrier-side regulation) -> OpenAVSwitch Carrier Board - Power
